Commit message: Added the slam SLAM_Pipeline

File: rover_gazebosim/urdf/rover.urdf (robot description, URDF)
Before this commit: robot rover, 31 links, 30 joints
Joints:
- joint joint3: limit lower=-0.5 upper=0.3 effort=10000 velocity=1 -> lower=-0.1 upper=0.1 effort=10000 velocity=1
- joint joint4: limit lower=-0.5 upper=0.3 effort=10000 velocity=1 -> lower=-0.1 upper=0.1 effort=10000 velocity=1
- joint joint_root: origin xyz=0.276421885520658 -0.526119109974194 -0.213679693338444 rpy=0 0 3.1415926 -> xyz=0.276421885520658 -0.526119109974194 -0.213679693338444 rpy=0 0 0
- joint joint_sensor_laser: origin xyz=0.276421885520658 -0.526119109974194 0.413679693338444 rpy=0 0 3.1415926 -> xyz=0.276421885520658 -0.526119109974194 0.413679693338444 rpy=0 0 0
- joint wheel_joint_1: axis -0.6621 -0.060914 0.74694 -> 0.6621 0.060914 -0.74694
- joint wheel_joint_2: axis -0.6621 -0.060914 0.74694 -> 0.6621 0.060914 -0.74694
- joint wheel_joint_3: axis -0.6621 -0.060914 0.74694 -> 0.6621 0.060914 -0.74694
- joint wheel_joint_4: axis 0.6621 0.060914 -0.74694 -> -0.6621 -0.060914 0.74694
- joint wheel_joint_5: axis 0.6621 0.060914 -0.74694 -> -0.6621 -0.060914 0.74694
- joint wheel_joint_6: axis 0.6621 0.060914 -0.74694 -> -0.6621 -0.060914 0.74694
