Commit message: Complete with RTAB Map.

File: husarion_components_description/urdf/orbbec_astra.urdf.xacro (robot description, xacro)
@@ -86,5 +86,5 @@
     <link name="${component_name_underscore}depth_optical_frame" />
     <joint name="${component_name_underscore}depth_to_${component_name_underscore}depth_optical_joint" type="fixed">
-      <origin xyz="0.0 0.0 0.0" rpy="${-pi/2} 0.0 ${-pi/2}" />
+      <origin xyz="0.0 0.0 0.0" rpy="0.0 0.0 0.0" />
       <parent link="${component_name_underscore}depth_frame" />
       <child link="${component_name_underscore}depth_optical_frame" />
